File: pcb/tile/tile.kicad_sch (KiCad schematic)
At the start: 15 parts, among them IC1 THVD1420DR, J1 LED Strip, J2 UPDI, J5 12V, J6 RS-485 Jack, U1 ATtiny3224-X

Commit message: Updated to account for a bulk cap as well as a resistor on the LED data line
Parts:
- added C7: 865080342006, Garth:CAPAE530X550N, symbol Garth Libraries:865080342006
- added R3: 330, Resistor_SMD:R_0805_2012Metric_Pad1.20x1.40mm_HandSolder, symbol Device:R_US
Connections:
- net +12V: now also C7.1 (+)
- net GND: now also C7.2 (-)
- net LED_Data: now also R3.1; no longer J1.2 (Pin_2)
- new net: J1.2 (Pin_2), R3.2
Other:
- note removed: "TODO: Add 100-470uF bulk caps"
- note removed: "TODO: Add series 330-470ohm resistor to LED_Data to dampen ringing"
- moved on the sheet: J1, J2, J5
