File: pcb/tile/tile.kicad_sch (KiCad schematic)
At the start: 17 parts, among them IC1 THVD1420DR, J1 LED Strip, J2 UPDI, J5 12V, J6 RS-485 Jack, U1 ATtiny3224-X

Commit message: pcb: 3.3V transceiver supply, second Row Bus chain, fab outputs
The THVD1420DR transceivers ran at VCC=5V while driving 3.3V-only GPIOs on
both boards. Per the datasheet the receiver output swings to VCC-0.4V min
(~4.6-4.8V at 5V), and the RX pull-ups went to 5V as well, so both the Pi's
and the RP2350's inputs sat out of spec. Both boards were bodged to 3.3V on
the bench; these schematics bring the sources in line.

pi-hat:
- IC3 supply, decoupling and RX pull-up moved from +5V to +3V3; no +5V net
  remains on the board.
- Second Row Bus chain added (IC4) so the 8 rows split across two chains -
  see docs/row-bus-protocol.md for why one chain no longer fits the frame
  budget. Chain A on uart0 (GPIO14/15), chain B on uart2 (GPIO4/5).
- Both direction lines moved onto the UARTs' own RTS pins, GPIO17 and
  GPIO7, so the kernel's RS-485 mode can eventually drive them with
  hardware timing instead of the host's busy-wait.
- Single RJ45 carries both chains on correctly-paired T568B conductors:
  chain A on pins 1-2, chain B on 3-6, grounds on the blue and brown pairs.

row-controller:
- Both transceivers, the INA220 and its I2C pull-ups moved to +3V3. +5V now
  only feeds the Xiao's VUSB input and the regulator that makes it.
- INA220 VBUS now senses +12V through the 5 mOhm shunt, matching what
  docs/row-bus-protocol.md's POWER command has always claimed it measures;
  it previously sat on the 5V rail and reported ~4.8V.

Also adds v1.0/1.2 gerbers and BOM CSVs, following the existing
gerber-1.1 pattern.

Reviewed the pi-hat netlist in detail - header pins, transceiver
orientation, rails, termination and pairing all check out. The
row-controller and tile changes are carried as-is.

Co-Authored-By: Claude Opus 5 <noreply@anthropic.com>
Parts:
- removed C6: 100nF, Capacitor_SMD:C_0805_2012Metric_Pad1.18x1.45mm_HandSolder, symbol Device:C
- C5: value 100nF -> 0.1uF
- U1: Manufacturer Name (none) -> Microchip Technology; Manufacturer Part Number (none) -> ATTINY3224-XF; Mouser Part Number (none) -> 579-ATTINY3224-XF; Mouser Price/Stock (none) -> https://www.mouser.com/en/ProductDetail/579-ATTINY3224-XF
Changed lines of the file:
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@@
 	(rectangle
 		(start 34.798 126.492)
-		(end 131.826 172.72)
+		(end 121.92 172.72)
 		(stroke
 			(width 0)
@@
 	)
 	(junction
-		(at 107.95 157.48)
-		(diameter 0)
-		(color 0 0 0 0)
-	)
-	(junction
 		(at 170.18 96.52)
 		(diameter 0)
@@
 	)
 	(junction
-		(at 107.95 137.16)
-		(diameter 0)
-		(color 0 0 0 0)
-	)
-	(junction
 		(at 80.01 76.2)
 		(diameter 0)
@@
 	(wire
 		(pts
-			(xy 120.65 148.59) (xy 120.65 157.48)
-		)
-		(stroke
-			(width 0)
-			(type default)
-		)
-	)
-	(wire
-		(pts
 			(xy 60.96 149.86) (xy 64.77 149.86)
 		)
@@
 	(wire
 		(pts
-			(xy 120.65 140.97) (xy 120.65 137.16)
-		)
-		(stroke
-			(width 0)
-			(type default)
-		)
-	)
-	(wire
-		(pts
 			(xy 39.37 97.79) (xy 46.99 97.79)
 		)
@@
 	(wire
 		(pts
-			(xy 120.65 157.48) (xy 107.95 157.48)
-		)
-		(stroke
-			(width 0)
-			(type default)
-		)
-	)
-	(wire
-		(pts
 			(xy 198.12 40.64) (xy 195.58 40.64)
 		)
@@
 	(wire
 		(pts
-			(xy 120.65 137.16) (xy 107.95 137.16)
-		)
-		(stroke
-			(width 0)
-			(type default)
-		)
-	)
-	(wire
-		(pts
 			(xy 195.58 40.64) (xy 195.58 44.45)
 		)
@@
 	)
 	(symbol
-		(lib_id "Device:C")
-		(at 120.65 144.78 0)
-		(unit 1)
-		(body_style 1)
-		(exclude_from_sim no)
-		(in_bom yes)
-		(on_board yes)
-		(in_pos_files yes)
-		(dnp no)
-		(fields_autoplaced yes)
-		(property "Reference" "C6"
-			(at 124.46 143.5099 0)
-			(show_name no)
-			(do_not_autoplace no)
-			(effects
-				(font
-					(size 1.27 1.27)
-				)
-				(justify left)
-			)
-		)
-		(property "Value" "100nF"
-			(at 124.46 146.0499 0)
-			(show_name no)
-			(do_not_autoplace no)
-			(effects
-				(font
-					(size 1.27 1.27)
-				)
-				(justify left)
-			)
-		)
-		(property "Footprint" "Capacitor_SMD:C_0805_2012Metric_Pad1.18x1.45mm_HandSolder"
-			(at 121.6152 148.59 0)
-			(hide yes)
-			(show_name no)
-			(do_not_autoplace no)
-			(effects
-				(font
-					(size 1.27 1.27)
-				)
-			)
-		)
-		(property "Datasheet" ""
-			(at 120.65 144.78 0)
-			(hide yes)
-			(show_name no)
-			(do_not_autoplace no)
-			(effects
-				(font
-					(size 1.27 1.27)
-				)
-			)
-		)
-		(property "Description" "Unpolarized capacitor"
-			(at 120.65 144.78 0)
-			(hide yes)
-			(show_name no)
-			(do_not_autoplace no)
-			(effects
-				(font
-					(size 1.27 1.27)
-				)
-			)
-		)
-		(pin "1"
-		)
-		(pin "2"
-		)
-		(instances
-			(project "tile"
-				(path "/68eea85a-4a75-40a0-9423-1988556e9fbf"
-					(reference "C6")
-					(unit 1)
-				)
-			)
-		)
-	)
-	(symbol
 		(lib_id "THVD1420DR:THVD1420DR")
 		(at 64.77 149.86 0)
@@
 			)
 		)
-		(property "Value" "100nF"
+		(property "Value" "0.1uF"
 			(at 111.76 146.0499 0)
 			(show_name no)
@@
 			(at 80.01 95.25 0)
 			(hide yes)
+			(show_name no)
+			(do_not_autoplace no)
+			(effects
+				(font
+					(size 1.27 1.27)
+				)
+			)
+		)
+		(property "Manufacturer Name" "Microchip Technology"
+			(at 80.01 95.25 0)
+			(hide yes)
+			(show_name no)
+			(do_not_autoplace no)
+			(effects
+				(font
+					(size 1.27 1.27)
+				)
+			)
+		)
+		(property "Manufacturer Part Number" "ATTINY3224-XF"
+			(at 80.01 95.25 0)
+			(hide yes)
+			(show_name no)
+			(do_not_autoplace no)
+			(effects
+				(font
+					(size 1.27 1.27)
+				)
+			)
+		)
+		(property "Mouser Part Number" "579-ATTINY3224-XF"
+			(at 80.01 95.25 0)
+			(hide yes)
+			(show_name no)
+			(do_not_autoplace no)
+			(effects
+				(font
+					(size 1.27 1.27)
+				)
+			)
+		)
+		(property "Mouser Price/Stock" "https://www.mouser.com/en/ProductDetail/579-ATTINY3224-XF"
+			(at 80.01 95.25 0)
+			(hide yes)
