File: pcb/row-controller/row-controller.kicad_sch (KiCad schematic)
At the start: 37 parts, among them IC1 INA220BIDGSR, IC2 THVD1420DR, IC3 THVD1420DR, J1 Power In, J2 5555140-2, J3 Power Row, J4 5555140-2, U1 XAIO ESP32-C3, U2 R-78E5.0-0.5

Commit message: Added a correction and a note to the schematic and design.
Other:
- note added: "TODO: Mount the RP2350 to the front side of the board. It will just clear the LDO and the power cap and save space"
Changed lines of the file:
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@@
+		)
+	)
+	(text "TODO: Mount the RP2350 to the\nfront side of the board. It will\njust clear the LDO and the power\ncap and save space"
+		(exclude_from_sim no)
+		(at 94.996 81.28 0)
+		(effects
+			(font
+				(size 1.27 1.27)
+			)
 		)
 	)
