File: pcb/row-controller/row-controller.kicad_sch (KiCad schematic)
At the start: 37 parts, among them IC1 INA220BIDGSR, IC2 THVD1420DR, IC3 THVD1420DR, J1 Power In, J2 5555140-2, J3 Power Row, J4 5555140-2, U1 XAIO ESP32-C3, U2 R-78E5.0-0.5

Commit message: pcb: 3.3V transceiver supply, second Row Bus chain, fab outputs
The THVD1420DR transceivers ran at VCC=5V while driving 3.3V-only GPIOs on
both boards. Per the datasheet the receiver output swings to VCC-0.4V min
(~4.6-4.8V at 5V), and the RX pull-ups went to 5V as well, so both the Pi's
and the RP2350's inputs sat out of spec. Both boards were bodged to 3.3V on
the bench; these schematics bring the sources in line.

pi-hat:
- IC3 supply, decoupling and RX pull-up moved from +5V to +3V3; no +5V net
  remains on the board.
- Second Row Bus chain added (IC4) so the 8 rows split across two chains -
  see docs/row-bus-protocol.md for why one chain no longer fits the frame
  budget. Chain A on uart0 (GPIO14/15), chain B on uart2 (GPIO4/5).
- Both direction lines moved onto the UARTs' own RTS pins, GPIO17 and
  GPIO7, so the kernel's RS-485 mode can eventually drive them with
  hardware timing instead of the host's busy-wait.
- Single RJ45 carries both chains on correctly-paired T568B conductors:
  chain A on pins 1-2, chain B on 3-6, grounds on the blue and brown pairs.

row-controller:
- Both transceivers, the INA220 and its I2C pull-ups moved to +3V3. +5V now
  only feeds the Xiao's VUSB input and the regulator that makes it.
- INA220 VBUS now senses +12V through the 5 mOhm shunt, matching what
  docs/row-bus-protocol.md's POWER command has always claimed it measures;
  it previously sat on the 5V rail and reported ~4.8V.

Also adds v1.0/1.2 gerbers and BOM CSVs, following the existing
gerber-1.1 pattern.

Reviewed the pi-hat netlist in detail - header pins, transceiver
orientation, rails, termination and pairing all check out. The
row-controller and tile changes are carried as-is.

Co-Authored-By: Claude Opus 5 <noreply@anthropic.com>
Parts:
- removed C6, C7: 100nF, Capacitor_SMD:C_0805_2012Metric_Pad1.18x1.45mm_HandSolder, symbol Device:C
- removed J2, J4: 5555140-2, 5555140-2:55551402, symbol 5555140-2:5555140-2
- added J5: Row Bus Header, Garth:1548129, symbol Garth Libraries:1548129
- added J6: Tile Bus Header, Garth:TB003-500-P04BE, symbol Garth Libraries:TB003-500-P04BE
- C3, C8: value .1uF -> 0.1uF
- C4, C5: value 100nF -> 0.1uF
- J1: Manufacturer Name (none) -> JST; Manufacturer Part Number (none) -> S05B-PASK-2(LF)(SN); Mouser Part Number (none) -> 306-S05BPASK2LFSN; Mouser Price/Stock (none) -> https://www.mouser.com/en/ProductDetail/306-S2B-XH-ALFSN
- R1: Manufacturer Name (none) -> TT Electronics; Manufacturer Part Number (none) -> LRMAT2010-R005FT4; Mouser Part Number (none) -> 756-LRMAT2010R005FT4; Mouser Price/Stock (none) -> https://www.mouser.com/en/ProductDetail/756-LRMAT2010R005FT4
- R11: Manufacturer Name (none) -> Vishay; Manufacturer Part Number (none) -> CRCW120610R0FKEAHP; Mouser Part Number (none) -> 71-CRCW120610R0FKEAH; Mouser Price/Stock (none) -> https://www.mouser.com/en/ProductDetail/71-CRCW120610R0FKEAH
- R2, R5: value 10K -> 4.7K
- U1: value XAIO ESP32-C3 -> XAIO RP2350; Manufacturer Part Number (none) -> 102010550; Mouser Part Number (none) -> 713-102010550; Mouser Price/Stock (none) -> https://www.mouser.com/en/ProductDetail/Seeed-Studio/102010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
- U2: symbol Regulator_Switching:R-78E5.0-0.5 -> Converter_DCDC:R-78E5.0-0.5; Manufacturer Name (none) -> RECOM Power; Manufacturer Part Number (none) -> R-78E5.0-0.5; Mouser Part Number (none) -> 919-R-78E5.0-0.5; Mouser Price/Stock (none) -> https://www.mouser.com/en/ProductDetail/919-R-78E5.0-0.5
Connections:
- net +3V3: now also C3.2, C4.1, C5.1, IC1.1 (A1), IC1.2 (A0), IC1.6 (VS), IC2.8 (VCC), IC3.8 (VCC), R2.1, R4.1, R5.1, R7.1
- net +5V: no longer C3.2, C4.1, C5.1, IC1.1 (A1), IC1.2 (A0), IC1.6 (VS), IC2.8 (VCC), IC3.8 (VCC), R2.1, R4.1, R5.1, R7.1
- net GND: now also J5.1, J6.1
- net PI-RxD: now also U1.4 (D3); no longer U1.10 (D9)
- net PI-TxD: now also U1.10 (D9); no longer U1.11 (D10)
- net ROW-SENSE: now also J6.2
- net ROW-XDIR: now also U1.11 (D10); no longer U1.4 (D3)
- net PI-TRCV-A renamed PI-TRCV_P
- net PI-TRCV_P: now also J5.3
- net PI-TRCV-B renamed PI-TRCV_N
- net PI-TRCV_N: now also J5.2
- net ROW-TRCV-A renamed ROW-TRCV_P
- net ROW-TRCV_P: now also J6.4
- net ROW-TRCV-B renamed ROW-TRCV_N
- net ROW-TRCV_N: now also J6.3
Other:
- note added: "Status LEDs"
- note removed: "TODO: Mount the RP2350 to the front side of the board. It will just clear the LDO and the power cap and save space"
- note removed: "TODO: Re-home Pi TxD and RxD to be on better pins for the Xiao RP2350, likely D0/D1"
- moved on the sheet: C5, C8, C9, D1, D2, D3, R10, R8, R9, U1
