File: pcb/row-controller/row-controller.kicad_pcb (KiCad board)
At the start: 2 copper layers, 52.1 x 29.5 mm, 35 parts, among them IC1 INA220BIDGSR, IC2 THVD1420DR, IC3 THVD1420DR, J1 Power In, J3 Power Row, J5 Row Bus Header, J6 Tile Bus Header, U1 XAIO RP2350, U2 R-78E5.0-0.5

Commit message: Several changes while testing.
Primary is that 5v was being used as the power rail when 3V3 was needed on the Pi hat and row controller board, where the RPi5 and RP2350 are both 3V3 logic.  On the Pi Hat a second UART to RS-485 was also added to have dual buses, enabling 6.25 Gbps, given the RPi5 is limited to 3.125Mbps
Other:
- board text added: "2026-08-09 v1.3"
- board text removed: "2025-10-29 v1.2"

Commit message: Fixed trace length for sense resistor.
Ensure the traces to IN+ and IN- go directly to those pins.  Electrically IN+ and Vbus connect, and since they are adjacent, I mistakenly wired the sense resistor to Vbus, with a dog leg over to IN+.  Flip that so it goes directly to IN+ with a dog leg to Vbus.  This keeps the line lengths for IN+ and IN- short and equal.
Parts:
- IC1: value INA220BIDGSR -> INA226; footprint INA220BIDGSR:SOP50P490X110-10N -> Package_SO:TSSOP-10_3x3mm_P0.5mm
- moved J1 8.75 mm to (123.7, 103.1)
- moved J3 8.65 mm to (123.7, 111.8)
- moved R1 0.45 mm to (117.6, 107.8), turned to -90 degrees
- turned C3 to 180 degrees
Connections:
- C3 pad 1: GND -> +3V3
- C3 pad 2: +3V3 -> GND
Routing:
- net Vrow: track 43.6 -> 32.0 mm
- net +12V: track 13.4 -> 14.1 mm

Commit message: Committing all PCB changes.  Everything has been sent and received from fab
Parts:
- removed J1: Power In, Connector_JST:JST_XH_S2B-XH-A_1x02_P2.50mm_Horizontal
- removed J3: Power Row, Connector_JST:JST_XH_S2B-XH-A_1x02_P2.50mm_Horizontal
- added J7: ~, Garth:Quad Powerpole, F.Cu at (126.3, 108.0)
Routing:
- net Vrow: track 32.0 -> 23.2 mm
- net +12V: track 14.1 -> 7.03 mm
- net /PI-TxD: track 30.2 -> 33.8 mm, vias 0 -> 1
- net +3V3: track 110.0 -> 108.8 mm
- net /ROW-RxD: track 39.7 -> 38.5 mm
Other:
- board text added: "2026-08-26 v1.3"
- board text removed: "2026-08-09 v1.3"
